File: UtilKeeb.kicad_pcb (KiCad board)
At the start: 2 copper layers, 123 parts, among them SW1 SW_Push, SW10 SW_Push, SW11 SW_Push, SW12 SW_Push, SW13 SW_Push, SW14 SW_Push, SW15 SW_Push, SW16 SW_Push, SW17 SW_Push, SW18 SW_Push, SW19 SW_Push, SW2 SW_Push, SW20 SW_Push, SW21 SW_Push, SW22 SW_Push, SW23 SW_Push, SW24 SW_Push, SW25 SW_Push, SW26 SW_Push, SW27 SW_Push, SW28 SW_Push, SW29 SW_Push, SW3 SW_Push, SW30 SW_Push, SW31 SW_Push, SW32 SW_Push, SW33 SW_Push, SW34 SW_Push, SW35 SW_Push, SW36 SW_Push, SW37 SW_Push, SW38 SW_Push, SW39 SW_Push, SW4 SW_Push, SW40 SW_Push, SW41 SW_Push, SW42 SW_Push, SW43 SW_Push, SW44 SW_Push, SW45 SW_Push, SW46 SW_Push, SW47 SW_Push, SW48 SW_Push, SW49 SW_Push, SW5 SW_Push, SW50 SW_Push, SW51 SW_Push, SW52 SW_Push, SW53 SW_Push, SW54 SW_Push, SW55 SW_Push, SW56 SW_Push, SW57 SW_Push, SW58 SW_Push, SW59 SW_Push, SW6 SW_Push, SW60 SW_Push, SW7 SW_Push, SW8 SW_Push, SW9 SW_Push

Commit message: Update too tired to finish for today
Parts:
- added S2: choc_stab, PCM_marbastlib-xp-choc:STAB_choc_2u, F.Cu at (33.5, 78.6)
- added S3: choc_stab, PCM_marbastlib-mx:STAB_MX_P_6.25u, F.Cu at (11.8, 140.2)
- added SW61: SW_Push, PCM_marbastlib-mx:STAB_MX_2u, F.Cu at (278.9, 21.5)
- SW4: footprint marbastlib-mx:STAB_MX_2.25u -> PCM_marbastlib-mx:SW_MX_1u
- SW60: footprint PCM_marbastlib-mx:STAB_MX_2u -> PCM_marbastlib-mx:SW_MX_1u
- moved D60 244.9 mm to (259.8, 24.8), turned to 90 degrees
- moved D61 236.2 mm to (313.9, 81.8), turned to 90 degrees
- moved D49 233.4 mm to (202.7, 24.0), turned to 90 degrees
- moved D50 229.9 mm to (232.2, 43.5), turned to 90 degrees
- moved D57 227.2 mm to (240.7, 24.1), turned to 90 degrees
- moved D36 223.2 mm to (145.3, 24.1), turned to 90 degrees
- moved D45 214.2 mm to (183.4, 24.2), turned to 90 degrees
- moved D37 213.3 mm to (175.0, 43.5), turned to 90 degrees
- moved D51 209.2 mm to (217.2, 62.9), turned to 90 degrees
- moved D46 209.1 mm to (213.0, 43.3), turned to 90 degrees
- moved D59 206.9 mm to (255.2, 62.9), turned to 90 degrees
- moved D53 206.5 mm to (221.7, 23.9), turned to 90 degrees
- moved D54 206.3 mm to (251.4, 43.4), turned to 90 degrees
- moved D31 203.6 mm to (126.2, 24.5), turned to 90 degrees
- moved D41 196.4 mm to (164.4, 24.1), turned to 90 degrees
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Routing:
- net (no net): track 0.53 -> 0.00 mm
Other:
- board outline added: 29.3 x 11.3 mm
