File: _restore_backup_2026-09-01T10-50-55-651/UtilKeeb.kicad_pcb (KiCad board)
At the start: 2 copper layers, 123 parts, among them SW1 SW_Push, SW10 SW_Push, SW11 SW_Push, SW12 SW_Push, SW13 SW_Push, SW14 SW_Push, SW15 SW_Push, SW16 SW_Push, SW17 SW_Push, SW18 SW_Push, SW19 SW_Push, SW2 SW_Push, SW20 SW_Push, SW21 SW_Push, SW22 SW_Push, SW23 SW_Push, SW24 SW_Push, SW25 SW_Push, SW26 SW_Push, SW27 SW_Push, SW28 SW_Push, SW29 SW_Push, SW3 SW_Push, SW30 SW_Push, SW31 SW_Push, SW32 SW_Push, SW33 SW_Push, SW34 SW_Push, SW35 SW_Push, SW36 SW_Push, SW37 SW_Push, SW38 SW_Push, SW39 SW_Push, SW4 SW_Push, SW40 SW_Push, SW41 SW_Push, SW42 SW_Push, SW43 SW_Push, SW44 SW_Push, SW45 SW_Push, SW46 SW_Push, SW47 SW_Push, SW48 SW_Push, SW49 SW_Push, SW5 SW_Push, SW50 SW_Push, SW51 SW_Push, SW52 SW_Push, SW53 SW_Push, SW54 SW_Push, SW55 SW_Push, SW56 SW_Push, SW57 SW_Push, SW58 SW_Push, SW59 SW_Push, SW6 SW_Push, SW60 SW_Push, SW7 SW_Push, SW8 SW_Push, SW9 SW_Push

Commit message: Update after School
Parts:
- SW10, SW14, SW25, SW30, SW35, SW40: footprint marbastlib-mx:SW_MX_1.25u -> marbastlib-mx:SW_MX_1u
- moved SW54 330.3 mm to (73.2, 324.9)
- moved SW40 301.0 mm to (58.2, 294.8)
- moved SW42 297.3 mm to (58.2, 309.8)
- moved SW43 295.4 mm to (58.2, 324.9)
- moved SW32 288.2 mm to (43.1, 309.8)
- moved SW33 286.0 mm to (43.1, 324.9)
- moved SW50 281.8 mm to (73.2, 279.7)
- moved SW51 280.7 mm to (73.2, 294.8)
- moved SW30 277.0 mm to (43.1, 294.8)
- moved SW52 271.9 mm to (73.2, 309.8)
- moved SW59 271.0 mm to (92.6, 268.8)
- moved SW58 270.9 mm to (88.3, 249.6)
- moved SW22 263.8 mm to (28.1, 309.8)
- moved SW23 257.3 mm to (28.1, 324.9)
- moved SW35 245.3 mm to (58.2, 234.6)
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Connections:
- D4 pad 1: /Row3 -> unconnected-(D4-K-Pad1)
Routing:
- net (no net): track 0.53 -> 0.00 mm
