File: _restore_backup_2026-09-01T10-50-55-651/UtilKeeb.kicad_sch (KiCad schematic)
At the start: 124 parts, among them SW1 SW_Push, SW10 SW_Push, SW11 SW_Push, SW12 SW_Push, SW13 SW_Push, SW14 SW_Push, SW15 SW_Push, SW16 SW_Push, SW17 SW_Push, SW18 SW_Push, SW19 SW_Push, SW2 SW_Push, SW20 SW_Push, SW21 SW_Push, SW22 SW_Push, SW23 SW_Push, SW24 SW_Push, SW25 SW_Push, SW26 SW_Push, SW27 SW_Push, SW28 SW_Push, SW29 SW_Push, SW3 SW_Push, SW30 SW_Push, SW31 SW_Push, SW32 SW_Push, SW33 SW_Push, SW34 SW_Push, SW35 SW_Push, SW36 SW_Push, SW37 SW_Push, SW38 SW_Push, SW39 SW_Push, SW4 SW_Push, SW40 SW_Push, SW41 SW_Push, SW42 SW_Push, SW43 SW_Push, SW44 SW_Push, SW45 SW_Push, SW46 SW_Push, SW47 SW_Push, SW48 SW_Push, SW49 SW_Push, SW5 SW_Push, SW50 SW_Push, SW51 SW_Push, SW52 SW_Push, SW53 SW_Push, SW54 SW_Push, SW55 SW_Push, SW56 SW_Push, SW57 SW_Push, SW58 SW_Push, SW59 SW_Push, SW6 SW_Push, SW60 SW_Push, SW61 SW_Push, SW7 SW_Push, SW8 SW_Push, SW9 SW_Push

Commit message: Update after School
Parts:
- SW10, SW14, SW25, SW30, SW35, SW40: footprint marbastlib-mx:SW_MX_1.25u -> marbastlib-mx:SW_MX_1u
Connections:
- net Row3: no longer D4.1 (K)
Changed lines of the file:
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@@
 	)
 	(junction
-		(at 35.56 76.2)
-		(diameter 0)
-		(color 0 0 0 0)
-	)
-	(junction
 		(at 152.4 38.1)
 		(diameter 0)
@@
 	(wire
 		(pts
-			(xy 22.86 76.2) (xy 35.56 76.2)
-		)
-		(stroke
-			(width 0)
-			(type default)
-		)
-	)
-	(wire
-		(pts
 			(xy 50.8 25.4) (xy 50.8 38.1)
 		)
@@
 			)
 		)
-		(property "Footprint" "marbastlib-mx:SW_MX_1.25u"
+		(property "Footprint" "marbastlib-mx:SW_MX_1u"
 			(at 93.98 78.74 0)
 			(hide yes)
@@
 			)
 		)
-		(property "Footprint" "marbastlib-mx:SW_MX_1.25u"
+		(property "Footprint" "marbastlib-mx:SW_MX_1u"
 			(at 68.58 78.74 0)
 			(hide yes)
@@
 			)
 		)
-		(property "Footprint" "marbastlib-mx:SW_MX_1.25u"
+		(property "Footprint" "marbastlib-mx:SW_MX_1u"
 			(at 81.28 78.74 0)
 			(hide yes)
@@
 			)
 		)
-		(property "Footprint" "marbastlib-mx:SW_MX_1.25u"
+		(property "Footprint" "marbastlib-mx:SW_MX_1u"
 			(at 43.18 63.5 0)
 			(hide yes)
@@
 			)
 		)
-		(property "Footprint" "marbastlib-mx:SW_MX_1.25u"
+		(property "Footprint" "marbastlib-mx:SW_MX_1u"
 			(at 106.68 78.74 0)
 			(hide yes)
@@
 			)
 		)
-		(property "Footprint" "marbastlib-mx:SW_MX_1.25u"
+		(property "Footprint" "marbastlib-mx:SW_MX_1u"
 			(at 30.48 78.74 0)
 			(hide yes)
